File: KiCad/thumbs/Vbox_thumbs.kicad_sch (KiCad schematic)
At the start: 38 parts, among them J1 Conn_01x02, J2 DuPont Connector, J2 JTAG_TC2030, J4 Conn_01x06, J5 Conn_01x06, J6 Conn_01x10, J7 Conn_01x10, SW1 Boot, U1 XC6206, U2 X05A26H12G, U3 RP2040, U4 W25Q128JVS, Y1 12MHz

Commit message: mobo complete...?
Parts:
- removed J4, J5: Conn_01x06, Connector_JST:JST_PH_B6B-PH-SM4-TB_1x06-1MP_P2.00mm_Vertical, symbol Connector_Generic:Conn_01x06
- removed J6, J7: Conn_01x10, Connector_JST:JST_PH_B10B-PH-SM4-TB_1x10-1MP_P2.00mm_Vertical, symbol Connector_Generic:Conn_01x10
- added D3: GREEN, LED_SMD:LED_0805_2012Metric, symbol Device:LED_Small
- added R4: 470, Resistor_SMD:R_0402_1005Metric, symbol Device:R_Small
- added SW10, SW11, SW12, SW13, SW14, SW15, SW16, SW17, SW18, SW19, SW2, SW20, SW21, SW3, SW4, SW5, SW6, SW7, SW8, SW9: ~, Buttons:RanaTadpole, symbol ranatadpole:RanaTadpole
Connections:
- net A: now also SW20.1
- net B: now also SW13.1
- net C_DN: now also SW19.1
- net C_LT: now also SW17.1
- net C_RT: now also SW21.1
- net C_UP: now also SW18.1
- net DOWN: now also SW5.1
- net GND: now also D3.1 (K), SW10.2, SW11.2, SW12.2, SW13.2, SW14.2, SW15.2, SW16.2, SW17.2, SW18.2, SW19.2, SW2.2, SW20.2, SW21.2, SW3.2, SW4.2, SW5.2, SW6.2, SW7.2, SW8.2, SW9.2
- net L: now also SW3.1
- net LEFT: now also SW4.1
- net LS: now also SW11.1
- net M1: now also SW7.1
- net M2: now also SW8.1
- net MS: now also SW12.1
- net R: now also SW9.1
- net RIGHT: now also SW6.1
- net START: now also SW2.1
- net UP: now also SW16.1
- net X: now also SW14.1
- net Y: now also SW10.1
- net Z: now also SW15.1
- net INDEX2: no longer names the net of U3.14 (GPIO11)
- net M3: no longer names the net of U3.11 (GPIO8)
- net M4: no longer names the net of U3.12 (GPIO9)
- net M5: no longer names the net of U3.13 (GPIO10)
- net PINKY2 renamed PICO_LED
- net PICO_LED: now also R4.1
- net RIGHTSTART: no longer names the net of U3.41 (GPIO29/ADC3)
- net RING2: no longer names the net of U3.35 (GPIO23)
- net UP2: no longer names the net of U3.3 (GPIO1)
- new net: D3.2 (A), R4.2
- no-connect marks 0 -> 26
Other:
- note added: "Logos"
- note added: "Pico LED"
